File: pcb/1-power.kicad_sch (KiCad schematic)
At the start: 0 parts

Commit message: Phase 3: populate power sheet; descriptive net names
Power sheet: bench eFuse (TPS259470A) with UVLO/OVLO string and EN
clamp, TPS2116 bench-priority mux with VBUS snubber, 3.3 V and 2.83 V
TPS73701 LDOs. Notes on the string's tap voltages, eFuse setting pins
and every DNP part. Project symbol library with the TPS259470A and
TPS73701DCQ drawn from the datasheet pin tables.

Nets renamed to spelled-out names (IS_BENCH_POWERED, *_INVERTED for
active-low, FEEDBACK, VTERMINATOR, TERMINATOR_EN) across the schematic,
pinout page, parts list and power block page.

Co-Authored-By: Claude Opus 5.5 <noreply@anthropic.com>
Parts:
- added C101: 1uF 50V X7R, Capacitor_SMD:C_0805_2012Metric, symbol Device:C
- added C102, C108: 100nF 50V, Capacitor_SMD:C_0402_1005Metric, symbol Device:C
- added C103: 2.2nF, Capacitor_SMD:C_0402_1005Metric, symbol Device:C
- added C104: 1nF, Capacitor_SMD:C_0402_1005Metric, symbol Device:C
- added C105, C106, C110, C112: 1uF 25V, Capacitor_SMD:C_0402_1005Metric, symbol Device:C
- added C107: 4.7uF 25V, Capacitor_SMD:C_0805_2012Metric, symbol Device:C
- added C109: 22uF 25V, Capacitor_SMD:C_0805_2012Metric, symbol Device:C
- added C111, C113: 10uF 25V, Capacitor_SMD:C_0805_2012Metric, symbol Device:C
- added D101: SMF15CA, Diode_SMD:D_SMF, symbol Device:D_TVS
- added D102: BZT52C5V6, Diode_SMD:D_SOD-123, symbol Device:D_Zener
- added J101: Bench 5V, symbol Connector:Screw_Terminal_01x02
- added R101: 510k, Resistor_SMD:R_0402_1005Metric, symbol Device:R
- added R102, R108, R118: 39k, Resistor_SMD:R_0402_1005Metric, symbol Device:R
- added R103: 3.9k, Resistor_SMD:R_0402_1005Metric, symbol Device:R
- added R104: 150k, Resistor_SMD:R_0402_1005Metric, symbol Device:R
- added R105, R109: 10k, Resistor_SMD:R_0402_1005Metric, symbol Device:R
- added R106: 1.5k, Resistor_SMD:R_0402_1005Metric, symbol Device:R
- added R107, R111, R116: 100k, Resistor_SMD:R_0402_1005Metric, symbol Device:R
- added R110: 1R, Resistor_SMD:R_0603_1608Metric, symbol Device:R
- added R112, R117: 75k, Resistor_SMD:R_0402_1005Metric, symbol Device:R
- added R113: 47k, Resistor_SMD:R_0402_1005Metric, symbol Device:R
- added R114: 27k, Resistor_SMD:R_0402_1005Metric, symbol Device:R
- added R115: 1M, Resistor_SMD:R_0603_1608Metric, symbol Device:R
- added R119: 5.6k, Resistor_SMD:R_0402_1005Metric, symbol Device:R
- added R120: 33k, Resistor_SMD:R_0402_1005Metric, symbol Device:R
- added R121: 270R, Resistor_SMD:R_0603_1608Metric, symbol Device:R
- added TP101: BENCH+, TestPoint:TestPoint_Loop_D2.50mm_Drill1.0mm, symbol Connector:TestPoint
- added TP102: GND, TestPoint:TestPoint_Loop_D2.50mm_Drill1.0mm, symbol Connector:TestPoint
- added U101: TPS259470ARPWR, symbol scsi-adapter:TPS259470A
- added U102: TPS2116DRLR, Package_TO_SOT_SMD:SOT-583-8, symbol Power_Management:TPS2116DRL
- added U103, U104: TPS73701DCQR, Package_TO_SOT_SMD:SOT-223-6, symbol scsi-adapter:TPS73701DCQ
Connections:
- net BENCH_5V: now also C105.1, R107.1, U101.6 (OUT), U102.3 (VIN1), U102.5 (MODE)
- net VBUS: now also C106.1, R110.1, U102.6 (VIN2)
- new net: R102.2, R103.1
- new net: R104.2, R105.1
- new net: R106.1, U101.9 (ILM)
- new net: C107.1, R110.2
- new net: R118.2, R119.1
- new net: C104.1, U101.10 (ITIMER)
- new net: C103.1, U101.7 (DVDT)
- new net +3V3: C111.1, R109.1, R113.1, U103.2 (OUT)
- new net +5V_SYS: C108.1, C109.1, C110.1, R111.1, U102.2 (VOUT), U102.7 (VOUT), U103.1 (IN)
- new net BENCH_EFUSE_EN: D102.1 (K), R101.2, R102.1, U101.1 (EN/UVLO)
- new net BENCH_EFUSE_FAULT_INVERTED: U101.4 (~{FLT})
- new net BENCH_EFUSE_OV: R103.2, R104.1, U101.2 (OVLO)
- new net BENCH_RAW: C101.1, C102.1, D101.1 (A1), J101.1 (Pin_1), R101.1, TP101.1, U101.5 (IN)
- new net GND: C101.2, C102.2, C103.2, C104.2, C105.2, C106.2, C107.2, C108.2, C109.2, C110.2, C111.2, C112.2, C113.2, D101.2 (A2), D102.2 (A), J101.2 (Pin_2), R105.2, R106.2, R108.2, R112.2, R114.2, R115.2, R117.2, R120.2, R121.2, TP102.1, U101.8 (GND), U102.1 (GND), U103.3 (GND), U103.6 (GND), U104.3 (GND), U104.6 (GND)
- new net IS_BENCH_POWERED: R109.2, U102.8 (ST)
- new net LDO_3V3_EN: R111.2, R112.1, U103.5 (EN)
- new net LDO_3V3_FEEDBACK: R113.2, R114.1, R115.1, U103.4 (FB)
- new net LDO_TERMINATOR_EN: R116.2, R117.1, U104.5 (EN)
- new net LDO_TERMINATOR_FEEDBACK: R119.2, R120.1, U104.4 (FB)
- new net MUX_BENCH_DETECT: R107.2, R108.1, U102.4 (PR1)
- new net TERMPWR: C112.1, R116.1, U104.1 (IN)
- new net VTERMINATOR: C113.1, R118.1, R121.1, U104.2 (OUT)
- no-connect marks 0 -> 1
Other:
- note added: "0.07 V"
- note added: "1.12 V"
- note added: "1.15 V"
- note added: "1.42 V"
- note added: "2.83 V terminator rail (VTERMINATOR)"
- note added: "3.3 V logic rail"
- note added: "Bench 5 V input"
- note added: "DNP. Fit if the terminal sees hot-plug spikes above the eFuse's 28 V abs max (long leads, inductive supply)."
- note added: "Power mux (bench priority)"
- note added: "Powered from TERMPWR (SCSI-2 5.4.1). Vout = 1.204 x (44.6k + 33k) / 33k = 2.83 V (2.72-2.94 V worst case). R121 bleed keeps >= 10 mA load (TPS737 accuracy spec) and sinks current pushed in from the bus."
- note added: "R115 DNP: trim pad across R114. Fit ~1M if +3V3 measures low at bring-up (+55 mV)."
- note added: "Set the bench supply to 5.0 V (5.1 V max). eFuse: OVLO 5.35 V, UVLO 4.22 V, ILIM 2.22 A, auto-retry. String R101-R105: UV = 1.2 x 712.9k/202.9k, OV = 1.2 x 712.9k/160k. D102 keeps EN <= 6.5 V abs max on a 24 V mistake."
- note added: "TPS2116 priority mode: MODE tied to VIN1. PR1 (MUX_BENCH_DETECT) = 0.281 x VIN1, so the bench wins above ~3.6 V. ST (IS_BENCH_POWERED) is high while running on the bench. VBUS snubber R110 + C107 damps plug-in ringing (5.7 uF on VBUS total)."
- note added: "UVLO/OVLO string R101-R105 (712.9k total). Tap voltages at left are nominal for BENCH_RAW = 5.0 V (7.0 uA). EN/UVLO and OVLO share one threshold: 1.20 V rising, 1.09 V falling (typ; 1.183-1.223 / 1.076-1.116 V). BENCH_EFUSE_EN = BENCH_RAW x (R102..R105 = 202.9k) / 712.9k turns on above 1.20 x 712.9 / 202.9 = 4.22 V, off below 1.09 x 712.9 / 202.9 = 3.83 V. 1.42 V at 5.0 V: on, with 0.22 V margin.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"
- note added: "VBUS snubber (reduce USB cable ringing)"
- note added: "Vout = 1.204 x (R113 + R114) / R114 = 3.30 V. EN on above ~4.0 V (100k/75k). FEEDBACK: the LDO adjusts OUT until its FB pin sits at its 1.204 V reference, so the divider sets Vout."
- note added: "eFuse setting pins: C103 on DVDT: output turn-on slew, ~5.5 ms ramp to 5 V (limits inrush). R106 on ILM: current limit, 2.22 A (R = 3334 / I). C104 on ITIMER, DNP: overcurrent blanking timer (how long current may exceed the limit before the eFuse acts). Open = shortest. Fit ~1 nF (~0.84 ms) if normal load steps trip the limit (FAULT pulses at bring-up)."
- note removed: "Power (blocks/1-power.md, parts list §1) Bench 5 V terminal + test loops, bench eFuse TPS259470A (OVLO 5.35 V, ILIM 2.22 A, EN Zener), SMF15CA (DNP), TPS2116 priority mux (bench = VIN1) + VBUS snubber, +5V_SYS bulk, TPS73701 3.3 V (+3V3) and TPS73701 2.83 V terminator rail (VTERM, fed from TERMPWR). Global rails (power symbols): +5V_SYS, +3V3, VTERM, TERMPWR, GND."
