File: pcb/1-power.kicad_sch (KiCad schematic)
At the start: 43 parts, among them J101 Bench 5V, U101 TPS259470ARPWR, U102 TPS2116DRLR, U103 TPS73701DCQR, U104 TPS73701DCQR

Commit message: Phase 3: populate TERMPWR sheet; schematic generator in pcb/_gen
TERMPWR sheet: CC detection (LM393 against a CJ431 2.5 V shunt
reference divided to 0.653 V, with hysteresis), the active-low
TERMPWR enable node (comparators wired-OR with the bench-present
FET), and the TERMPWR eFuse with its OVLO-as-enable divider, jumper,
TVS and indicator LEDs. Includes the owner's CJ431 and PWR_FLAG notes.

pcb/_gen regenerates the generated sheets and checks them against
KiCad's netlist. It refuses to overwrite a sheet edited in KiCad
since the last build (content fingerprints). Adds a CJ431 symbol
with JCET's pinout, and restores the USB_HS net-class patterns that
a KiCad save had dropped.
Other:
- note added: "PWR_FLAG is not a part. It tells KiCad's ERC that a net is powered from outside the drawn symbols (the terminal, USB VBUS), so it doesn't report 'power input not driven'."
- note added: "eFuse setting pins: C103 on DVDT (dV/dt, output voltage slew rate): ~5.5 ms ramp to 5 V (limits inrush). R106 on ILM (I-limit: sets the current limit; the pin voltage is also a current monitor): 2.22 A (R = 3334 / I). C104 on ITIMER (I-timer), DNP: overcurrent blanking timer (how long current may exceed the limit before the eFuse acts). Open = shortest. Fit ~1 nF (~0.84 ms) if normal load steps t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"
- note removed: "eFuse setting pins: C103 on DVDT: output turn-on slew, ~5.5 ms ramp to 5 V (limits inrush). R106 on ILM: current limit, 2.22 A (R = 3334 / I). C104 on ITIMER, DNP: overcurrent blanking timer (how long current may exceed the limit before the eFuse acts). Open = shortest. Fit ~1 nF (~0.84 ms) if normal load steps trip the limit (FAULT pulses at bring-up)."
Changed lines of the file:
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@@
 	(wire (pts (xy 71.12 38.1) (xy 71.12 40.64)) (stroke (width 0) (type default)))
 	(label "BENCH_RAW" (at 71.12 40.64 0) (effects (font (size 1.27 1.27)) (justify left bottom)))
+	(text "PWR_FLAG is not a part. It tells KiCad's ERC that a net\nis powered from outside the drawn symbols (the terminal,\nUSB VBUS), so it doesn't report 'power input not driven'." (exclude_from_sim no) (at 66.04 48.26 0) (effects (font (size 1.016 1.016) (italic yes)) (justify left top)))
 	(symbol (lib_id "power:PWR_FLAG") (at 83.82 38.1 0) (unit 1) (exclude_from_sim no) (in_bom no) (on_board no) (dnp no)
 		(property "Reference" "#FLG102" (at 83.82 33.02 0) (effects (font (size 1.27 1.27)) (justify left) (hide yes)))
@@
 		(instances (project "scsi-adapter" (path "/2c5b21a9-7d0d-4304-8bd9-0602cba3b7b5/c5f4e78b-92c1-44f5-913e-e393dcfaf39d" (reference "#PWR110") (unit 1))))
 	)
-	(text "eFuse setting pins:\nC103 on DVDT: output turn-on slew,\n  ~5.5 ms ramp to 5 V (limits inrush).\nR106 on ILM: current limit, 2.22 A\n  (R = 3334 / I).\nC104 on ITIMER, DNP: overcurrent blanking\n  timer (how long current may exceed the\n  limit before the eFuse acts). Open =\n  shortest. Fit ~1 nF (~0.84 ms) if normal\n  load steps trip the limit (FAULT pulses\n  at bring-up)." (exclude_from_sim no) (at 172.72 83.82 0) (effects (font (size 1.016 1.016) (italic yes)) (justify left top)))
+	(text "eFuse setting pins:\nC103 on DVDT (dV/dt, output voltage slew\n  rate): ~5.5 ms ramp to 5 V (limits inrush).\nR106 on ILM (I-limit: sets the current limit;\n  the pin voltage is also a current monitor):\n  2.22 A (R = 3334 / I).\nC104 on ITIMER (I-timer), DNP: overcurrent\n  blanking timer (how long current may\n  exceed the limit before the eFuse acts).\n  Open = shortest. Fit ~1 nF (~0.84 ms) if normal\n  load steps trip the limit (FAULT pulses\n  at bring-up)." (exclude_from_sim no) (at 172.72 83.82 0) (effects (font (size 1.016 1.016) (italic yes)) (justify left top)))
 	(symbol (lib_id "Device:C") (at 193.04 132.08 0) (unit 1) (exclude_from_sim no) (in_bom yes) (on_board yes) (dnp no)
 		(property "Reference" "C105" (at 190.5 130.81 0) (effects (font (size 1.27 1.27)) (justify right)))

Commit message: Phase 3: footprint audit fixes and project footprint library
- New project footprint library pcb/scsi-adapter.pretty, generated by
  pcb/_gen/footprints.py from datasheet land patterns: TI RPW0010A (U101/U201),
  Kangnex WJ500V (J101), TE AMPLIMITE .050 HD50 (J302), SHOU HAN TF PUSH
  microSD (J501), Abracon AOTA-B201610 polarized inductor (L401), SHOU HAN
  2-pos DIP (SW301). fp-lib-table added.
- J303 LA header: 2x17 box header C20920, pins 33/34 NC (34-way ribbon to a
  future 2x16 adapter board).
- J302 HD50: TE 5787082-5 squeeze-latch receptacle; shielded symbol, shell to
  GND via R343 0R. TE STEP model git-ignored (pcb/scsi-adapter.3dshapes/).
- D101/D204/D605: D_SMF -> D_SOD-123F (parts are SOD-123FL).
- L401 pins swapped so pad 1 = polarity dot = DVDD_1V1 (RP2350 Fig. 23).
- SW401/SW402: Hroparts K2-1102DP C110153 on SW_PUSH_6mm.
- NOTES, decisions, sources updated; J601 pad question closed; RP2350B
  minimal-design layout copy planned (open question 17).
Parts:
- D101: footprint Diode_SMD:D_SMF -> Diode_SMD:D_SOD-123F
- J101: footprint (none) -> scsi-adapter:TerminalBlock_Kangnex_WJ500V-5.08-2P_1x02_P5.08mm_Horizontal
- U101: footprint (none) -> scsi-adapter:Texas_RPW0010A_VQFN-HR-10_2x2mm_P0.45mm
Changed lines of the file:
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@@
 		(property "Reference" "J101" (at 55.88 40.64 0) (effects (font (size 1.27 1.27)) (justify left)))
 		(property "Value" "Bench 5V" (at 55.88 52.07 0) (effects (font (size 1.27 1.27)) (justify left)))
-		(property "Footprint" "" (at 55.88 45.72 0) (effects (font (size 1.27 1.27)) (hide yes)))
+		(property "Footprint" "scsi-adapter:TerminalBlock_Kangnex_WJ500V-5.08-2P_1x02_P5.08mm_Horizontal" (at 55.88 45.72 0) (effects (font (size 1.27 1.27)) (hide yes)))
 		(property "Datasheet" "" (at 55.88 45.72 0) (effects (font (size 1.27 1.27)) (hide yes)))
-		(property "Description" "Kangnex WJ500V-5.08-2P, 5.08 mm. Footprint to do." (at 55.88 45.72 0) (effects (font (size 1.27 1.27)) (hide yes)))
+		(property "Description" "Kangnex WJ500V-5.08-2P, 5.08 mm" (at 55.88 45.72 0) (effects (font (size 1.27 1.27)) (hide yes)))
 		(property "LCSC" "C8465" (at 55.88 45.72 0) (effects (font (size 1.27 1.27)) (hide yes)))
 		(property "Fit" "Hand" (at 55.88 45.72 0) (effects (font (size 1.27 1.27)) (hide yes)))
@@
 		(property "Reference" "D101" (at 53.34 69.85 270) (effects (font (size 1.27 1.27)) (justify right)))
 		(property "Value" "SMF15CA" (at 53.34 72.39 270) (effects (font (size 1.27 1.27)) (justify right)))
-		(property "Footprint" "Diode_SMD:D_SMF" (at 50.8 71.12 0) (effects (font (size 1.27 1.27)) (hide yes)))
+		(property "Footprint" "Diode_SMD:D_SOD-123F" (at 50.8 71.12 0) (effects (font (size 1.27 1.27)) (hide yes)))
 		(property "Datasheet" "" (at 50.8 71.12 0) (effects (font (size 1.27 1.27)) (hide yes)))
 		(property "Description" "Bidirectional TVS, footprint only" (at 50.8 71.12 0) (effects (font (size 1.27 1.27)) (hide yes)))
@@
 		(property "Reference" "U101" (at 139.7 41.91 0) (effects (font (size 1.27 1.27)) (justify left)))
 		(property "Value" "TPS259470ARPWR" (at 170.18 41.91 0) (effects (font (size 1.27 1.27)) (justify right)))
-		(property "Footprint" "" (at 154.94 50.8 0) (effects (font (size 1.27 1.27)) (hide yes)))
+		(property "Footprint" "scsi-adapter:Texas_RPW0010A_VQFN-HR-10_2x2mm_P0.45mm" (at 154.94 50.8 0) (effects (font (size 1.27 1.27)) (hide yes)))
 		(property "Datasheet" "https://www.ti.com/lit/ds/symlink/tps25947.pdf" (at 154.94 50.8 0) (effects (font (size 1.27 1.27)) (hide yes)))
-		(property "Description" "Bench eFuse. RPW QFN-10 footprint to do." (at 154.94 50.8 0) (effects (font (size 1.27 1.27)) (hide yes)))
+		(property "Description" "Bench eFuse" (at 154.94 50.8 0) (effects (font (size 1.27 1.27)) (hide yes)))
 		(property "LCSC" "C3662799" (at 154.94 50.8 0) (effects (font (size 1.27 1.27)) (hide yes)))
 		(property "Fit" "JLC" (at 154.94 50.8 0) (effects (font (size 1.27 1.27)) (hide yes)))

Commit message: good chunk of power routing
Parts:
- removed TP101: BENCH+, TestPoint:TestPoint_Loop_D2.50mm_Drill1.0mm, symbol Connector:TestPoint
- removed TP102: GND, TestPoint:TestPoint_Loop_D2.50mm_Drill1.0mm, symbol Connector:TestPoint

Commit message: sch update
Parts:
- added C114: 1uF 25V, Capacitor_SMD:C_0402_1005Metric, symbol Device:C
Connections:
- net BENCH_5V: now also C114.1
- net GND: now also C114.2
Changed lines of the file:
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@@
 		)
 	)
+	(symbol (lib_id "Device:C") (at 264.16 121.92 0) (unit 1) (exclude_from_sim no) (in_bom yes) (on_board yes) (dnp no)
+		(property "Reference" "C114" (at 261.62 120.65 0) (effects (font (size 1.27 1.27)) (justify right)))
+		(property "Value" "1uF 25V" (at 261.62 123.19 0) (effects (font (size 1.27 1.27)) (justify right)))
+		(property "Footprint" "Capacitor_SMD:C_0402_1005Metric" (at 264.16 121.92 0) (effects (font (size 1.27 1.27)) (hide yes)))
+		(property "Datasheet" "" (at 264.16 121.92 0) (effects (font (size 1.27 1.27)) (hide yes)))
+		(property "Description" "VIN1: place at U102 pin 3" (at 264.16 121.92 0) (effects (font (size 1.27 1.27)) (hide yes)))
+		(property "LCSC" "C52923" (at 264.16 121.92 0) (effects (font (size 1.27 1.27)) (hide yes)))
+		(property "Fit" "JLC" (at 264.16 121.92 0) (effects (font (size 1.27 1.27)) (hide yes)))
+		(pin "1")
+		(pin "2")
+		(instances (project "scsi-adapter" (path "/2c5b21a9-7d0d-4304-8bd9-0602cba3b7b5/c5f4e78b-92c1-44f5-913e-e393dcfaf39d" (reference "C114") (unit 1))))
+	)
+	(wire (pts (xy 264.16 118.11) (xy 264.16 115.57)) (stroke (width 0) (type default)))
+	(hierarchical_label "BENCH_5V" (shape output) (at 264.16 115.57 0) (effects (font (size 1.27 1.27)) (justify left)))
+	(wire (pts (xy 264.16 125.73) (xy 264.16 128.27)) (stroke (width 0) (type default)))
+	(symbol (lib_id "power:GND") (at 264.16 128.27 0) (unit 1) (exclude_from_sim no) (in_bom no) (on_board no) (dnp no)
+		(property "Reference" "#PWR152" (at 264.16 128.27 0) (effects (font (size 1.27 1.27)) (justify left) (hide yes)))
+		(property "Value" "GND" (at 264.16 133.35 0) (effects (font (size 1.27 1.27))))
+		(property "Footprint" "" (at 264.16 128.27 0) (effects (font (size 1.27 1.27)) (hide yes)))
+		(property "Datasheet" "" (at 264.16 128.27 0) (effects (font (size 1.27 1.27)) (hide yes)))
+		(property "Description" "" (at 264.16 128.27 0) (effects (font (size 1.27 1.27)) (hide yes)))
+		(pin "1")
+		(instances (project "scsi-adapter" (path "/2c5b21a9-7d0d-4304-8bd9-0602cba3b7b5/c5f4e78b-92c1-44f5-913e-e393dcfaf39d" (reference "#PWR152") (unit 1))))
+	)
 )
