File: pcb/1-power.kicad_sch (KiCad schematic)
At the start: 42 parts, among them J101 Bench 5V, U101 TPS259470ARPWR, U102 TPS2116DRLR, U103 TPS73701DCQR, U104 TPS73701DCQR

Commit message: Swap ten preferred parts for basic ones; regenerate JLC order files
R101 510k becomes 0603 C23192 (the 0402 C11616 ran out at JLC). Nine more
preferred lines are replaced so JLC's BOM tool lists them as basic:
- same-ratio pairs: LDO EN dividers 20k/15k, TPS2116 PR1 51k/20k
- re-valued pairs: bench string R2 33k + 10k, TERMPWR R_ILM 2.2k + 510R (1.23 A),
  TERMPWR UVLO 51k/20k (4.26 V), 3.3 V LDO R2 = 33k || 150k on the former trim pad R115
- 0603 for the same value: R104, R118, R119, R215, C103, C204
Sheets, generator scripts, PCB (owner's re-layout, silkscreen stripped from the new
0603 parts, fields synced), docs and pcb/fab are updated. DRC clean on the saved board.
Parts:
- C103: footprint Capacitor_SMD:C_0402_1005Metric -> Capacitor_SMD:C_0603_1608Metric; LCSC C1531 -> C1604
- R101: footprint Resistor_SMD:R_0402_1005Metric -> Resistor_SMD:R_0603_1608Metric; LCSC C11616 -> C23192
- R102: value 39k -> 33k; LCSC C25783 -> C25779
- R103: value 3.9k -> 10k; LCSC C51721 -> C25744
- R104: footprint Resistor_SMD:R_0402_1005Metric -> Resistor_SMD:R_0603_1608Metric; LCSC C25755 -> C22807
- R107: value 100k -> 51k; LCSC C25741 -> C25794
- R108: value 39k -> 20k; LCSC C25783 -> C25765
- R111, R116: value 100k -> 20k; LCSC C25741 -> C25765
- R112, R117: value 75k -> 15k; LCSC C25798 -> C25756
- R114: value 27k -> 33k; LCSC C25771 -> C25779
- R115: value 1M -> 150k; Fit DNP -> JLC; LCSC (none) -> C22807; now fitted
- R118: footprint Resistor_SMD:R_0402_1005Metric -> Resistor_SMD:R_0603_1608Metric; LCSC C25783 -> C23153
- R119: footprint Resistor_SMD:R_0402_1005Metric -> Resistor_SMD:R_0603_1608Metric; LCSC C25908 -> C23189
Other:
- note added: "1.19 V"
- note added: "R115 across R114: 33k || 150k = 27.05k (no basic 27k in 0402). Was a DNP trim pad until 2026-10-14."
- note added: "Set the bench supply to 5.0 V (5.1 V max). eFuse: OVLO 5.35 V, UVLO 4.21 V, ILIM 2.22 A, auto-retry. String R101-R105: UV = 1.2 x 713k/203k, OV = 1.2 x 713k/160k. D102 keeps EN <= 6.5 V abs max on a 24 V mistake."
- note added: "TPS2116 priority mode: MODE tied to VIN1. PR1 (MUX_BENCH_DETECT) = 0.282 x VIN1, so the bench wins above ~3.6 V. ST (IS_BENCH_POWERED) is high while running on the bench. VBUS snubber R110 + C107 damps plug-in ringing (5.7 uF on VBUS total)."
- note added: "UVLO/OVLO string R101-R105 (713k total). Tap voltages at left are nominal for BENCH_RAW = 5.0 V (7.0 uA). EN/UVLO and OVLO share one threshold: 1.20 V rising, 1.09 V falling (typ; 1.183-1.223 / 1.076-1.116 V). BENCH_EFUSE_EN = BENCH_RAW x (R102..R105 = 203k) / 713k turns on above 1.20 x 713 / 203 = 4.21 V, off below 1.09 x 713 / 203 = 3.83 V. 1.42 V at 5.0 V: on, with 0.22 V margin. BENCH_EFUSE_O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"
- note added: "Vout = 1.204 x (R113 + R2) / R2 = 3.30 V, R2 = R114 || R115 = 27.05k. EN on above ~4.0 V (20k/15k). FEEDBACK: the LDO adjusts OUT until its FB pin sits at its 1.204 V reference, so the divider sets Vout."
- note removed: "1.15 V"
- note removed: "R115 DNP: trim pad across R114. Fit ~1M if +3V3 measures low at bring-up (+55 mV)."
- note removed: "Set the bench supply to 5.0 V (5.1 V max). eFuse: OVLO 5.35 V, UVLO 4.22 V, ILIM 2.22 A, auto-retry. String R101-R105: UV = 1.2 x 712.9k/202.9k, OV = 1.2 x 712.9k/160k. D102 keeps EN <= 6.5 V abs max on a 24 V mistake."
- note removed: "TPS2116 priority mode: MODE tied to VIN1. PR1 (MUX_BENCH_DETECT) = 0.281 x VIN1, so the bench wins above ~3.6 V. ST (IS_BENCH_POWERED) is high while running on the bench. VBUS snubber R110 + C107 damps plug-in ringing (5.7 uF on VBUS total)."
- note removed: "UVLO/OVLO string R101-R105 (712.9k total). Tap voltages at left are nominal for BENCH_RAW = 5.0 V (7.0 uA). EN/UVLO and OVLO share one threshold: 1.20 V rising, 1.09 V falling (typ; 1.183-1.223 / 1.076-1.116 V). BENCH_EFUSE_EN = BENCH_RAW x (R102..R105 = 202.9k) / 712.9k turns on above 1.20 x 712.9 / 202.9 = 4.22 V, off below 1.09 x 712.9 / 202.9 = 3.83 V. 1.42 V at 5.0 V: on, with 0.22 V margin.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"
- note removed: "Vout = 1.204 x (R113 + R114) / R114 = 3.30 V. EN on above ~4.0 V (100k/75k). FEEDBACK: the LDO adjusts OUT until its FB pin sits at its 1.204 V reference, so the divider sets Vout."
Changed lines of the file:
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@@
 		)
 	)
-	(text "R115 DNP: trim pad across R114. Fit ~1M if\n+3V3 measures low at bring-up (+55 mV)."
+	(text "R115 across R114: 33k || 150k = 27.05k (no basic\n27k in 0402). Was a DNP trim pad until 2026-10-14."
 		(exclude_from_sim no)
 		(at 137.16 233.68 0)
@@
 		)
 	)
-	(text "Set the bench supply to 5.0 V (5.1 V max). eFuse: OVLO 5.35 V, UVLO 4.22 V, ILIM 2.22 A, auto-retry.\nString R101-R105: UV = 1.2 x 712.9k/202.9k, OV = 1.2 x 712.9k/160k. D102 keeps EN <= 6.5 V abs max on a 24 V mistake."
+	(text "Set the bench supply to 5.0 V (5.1 V max). eFuse: OVLO 5.35 V, UVLO 4.21 V, ILIM 2.22 A, auto-retry.\nString R101-R105: UV = 1.2 x 713k/203k, OV = 1.2 x 713k/160k. D102 keeps EN <= 6.5 V abs max on a 24 V mistake."
 		(exclude_from_sim no)
 		(at 20.32 24.82 0)
@@
 		)
 	)
-	(text "UVLO/OVLO string R101-R105 (712.9k total). Tap voltages at left are nominal for BENCH_RAW = 5.0 V (7.0 uA).\nEN/UVLO and OVLO share one threshold: 1.20 V rising, 1.09 V falling (typ; 1.183-1.223 / 1.076-1.116 V).\nBENCH_EFUSE_EN = BENCH_RAW x (R102..R105 = 202.9k) / 712.9k\n    turns on above 1.20 x 712.9 / 202.9 = 4.22 V, off below 1.09 x 712.9 / 202.9 = 3.83 V.\n    1.42 V at 5.0 V: on, with 0.22 V margin.\nBENCH_EFUSE_OV = BENCH_RAW x (R104 + R105 = 160k) / 712.9k\n    trips off above 1.20 x 712.9 / 160 = 5.35 V, recovers below 1.09 x 712.9 / 160 = 4.86 V.\n    1.12 V at 5.0 V: 78 mV under the trip, but inside the hysteresis band, so after a trip\n    the bench must come back below 4.86 V before the eFuse turns on again.\nWorst case (thresholds, 1 % R, +-0.1 uA pin leakage): UV 4.05-4.41 V, OV 5.14-5.59 V.\nR102 + R103 = 42.9k and R104 + R105 = 160k: no 43k or 160k 0402 1 % part is JLC basic/preferred,\n    so each is two no-fee parts. The unlabelled joints carry no function.\nR101 = 510k keeps the string >= 350k (TI's reverse-polarity guidance). Much bigger and the\n    +-0.1 uA pin leakage moves the OV trip enough to break the 5.5 V limit (NOTES, R059/R061)."
+	(text "UVLO/OVLO string R101-R105 (713k total). Tap voltages at left are nominal for BENCH_RAW = 5.0 V (7.0 uA).\nEN/UVLO and OVLO share one threshold: 1.20 V rising, 1.09 V falling (typ; 1.183-1.223 / 1.076-1.116 V).\nBENCH_EFUSE_EN = BENCH_RAW x (R102..R105 = 203k) / 713k\n    turns on above 1.20 x 713 / 203 = 4.21 V, off below 1.09 x 713 / 203 = 3.83 V.\n    1.42 V at 5.0 V: on, with 0.22 V margin.\nBENCH_EFUSE_OV = BENCH_RAW x (R104 + R105 = 160k) / 713k\n    trips off above 1.20 x 713 / 160 = 5.35 V, recovers below 1.09 x 713 / 160 = 4.86 V.\n    1.12 V at 5.0 V: 78 mV under the trip, but inside the hysteresis band, so after a trip\n    the bench must come back below 4.86 V before the eFuse turns on again.\nWorst case (thresholds, 1 % R, +-0.1 uA pin leakage): UV 4.05-4.41 V, OV 5.14-5.59 V.\nR102 + R103 = 43k (33k + 10k) and R104 + R105 = 160k (150k 0603 + 10k): no 43k or 160k part is JLC basic,\n    so each is two basic parts. The unlabelled joints carry no function.\nR101 = 510k keeps the string >= 350k (TI's reverse-polarity guidance). Much bigger and the\n    +-0.1 uA pin leakage moves the OV trip enough to break the 5.5 V limit (NOTES, R059/R061)."
 		(exclude_from_sim no)
 		(at 20.32 104.14 0)
@@
 		)
 	)
-	(text "Vout = 1.204 x (R113 + R114) / R114 = 3.30 V. EN on above ~4.0 V (100k/75k).\nFEEDBACK: the LDO adjusts OUT until its FB pin sits at its 1.204 V reference, so the divider sets Vout."
+	(text "Vout = 1.204 x (R113 + R2) / R2 = 3.30 V, R2 = R114 || R115 = 27.05k. EN on above ~4.0 V (20k/15k).\nFEEDBACK: the LDO adjusts OUT until its FB pin sits at its 1.204 V reference, so the divider sets Vout."
 		(exclude_from_sim no)
 		(at 20.32 169.6 0)
@@
 		)
 	)
-	(text "TPS2116 priority mode: MODE tied to VIN1. PR1 (MUX_BENCH_DETECT) = 0.281 x VIN1, so the bench wins above ~3.6 V.\nST (IS_BENCH_POWERED) is high while running on the bench. VBUS snubber R110 + C107 damps plug-in ringing (5.7 uF on VBUS total)."
+	(text "TPS2116 priority mode: MODE tied to VIN1. PR1 (MUX_BENCH_DETECT) = 0.282 x VIN1, so the bench wins above ~3.6 V.\nST (IS_BENCH_POWERED) is high while running on the bench. VBUS snubber R110 + C107 damps plug-in ringing (5.7 uF on VBUS total)."
 		(exclude_from_sim no)
 		(at 226.06 24.82 0)
@@
 		)
 	)
-	(text "1.15 V"
+	(text "1.19 V"
 		(exclude_from_sim no)
 		(at 115.57 104.775 0)
@@
 			)
 		)
-		(property "Footprint" "Resistor_SMD:R_0402_1005Metric"
+		(property "Footprint" "Resistor_SMD:R_0603_1608Metric"
 			(at 335.28 205.74 0)
 			(effects
@@
 			)
 		)
-		(property "LCSC" "C25783"
+		(property "LCSC" "C23153"
 			(at 335.28 205.74 0)
 			(effects
@@
 			)
 		)
-		(property "Value" "75k"
+		(property "Value" "15k"
 			(at 45.72 219.71 0)
 			(effects
@@
 			)
 		)
-		(property "LCSC" "C25798"
+		(property "LCSC" "C25756"
 			(at 48.26 218.44 0)
 			(effects
@@
 			)
 		)
-		(property "Footprint" "Resistor_SMD:R_0402_1005Metric"
+		(property "Footprint" "Resistor_SMD:R_0603_1608Metric"
 			(at 335.28 218.44 0)
 			(effects
@@
 			)
 		)
-		(property "LCSC" "C25908"
+		(property "LCSC" "C23189"
 			(at 335.28 218.44 0)
 			(effects
@@
 			)
 		)
-		(property "Footprint" "Resistor_SMD:R_0402_1005Metric"
+		(property "Footprint" "Resistor_SMD:R_0603_1608Metric"
 			(at 127 86.36 0)
 			(effects
@@
 			)
 		)
-		(property "LCSC" "C11616"
+		(property "LCSC" "C23192"
 			(at 127 86.36 0)
 			(effects
@@
 			)
 		)
-		(property "Value" "3.9k"
+		(property "Value" "10k"
 			(at 124.46 113.03 0)
 			(effects
@@
 			)
 		)
-		(property "Description" "String R2 (39k + 3.9k)"
+		(property "Description" "String R2 (33k + 10k)"
 			(at 127 111.76 0)
 			(effects
@@
 			)
 		)
-		(property "LCSC" "C51721"
+		(property "LCSC" "C25744"
 			(at 127 111.76 0)
 			(effects
@@
 			)
 		)
-		(property "Value" "39k"
+		(property "Value" "20k"
 			(at 238.76 102.87 0)
 			(effects
@@
 			)
 		)
-		(property "LCSC" "C25783"
+		(property "LCSC" "C25765"
 			(at 241.3 101.6 0)
 			(effects
@@
 			)
 		)
-		(property "Footprint" "Capacitor_SMD:C_0402_1005Metric"
+		(property "Footprint" "Capacitor_SMD:C_0603_1608Metric"
 			(at 142.24 67.31 0)
 			(effects
@@
 			)
 		)
-		(property "LCSC" "C1531"
+		(property "LCSC" "C1604"
 			(at 142.24 67.31 0)
 			(effects
@@
 			)
 		)
-		(property "Value" "27k"
+		(property "Value" "33k"
 			(at 109.22 219.71 0)
 			(effects
@@
 			)
 		)
-		(property "Description" "FB R2"
+		(property "Description" "FB R2 (33k || R115 150k)"
 			(at 111.76 218.44 0)
 			(effects
@@
 			)
 		)
-		(property "LCSC" "C25771"
+		(property "LCSC" "C25779"
 			(at 111.76 218.44 0)
 			(effects
@@
 			)
 		)
-		(property "Value" "75k"
+		(property "Value" "15k"
 			(at 254 219.71 0)
 			(effects
@@
 			)
 		)
-		(property "LCSC" "C25798"
+		(property "LCSC" "C25756"
 			(at 256.54 218.44 0)
 			(effects
@@
 			)
 		)
-		(property "Value" "100k"
+		(property "Value" "20k"
 			(at 254 207.01 0)
 			(effects
@@
 			)
 		)
-		(property "LCSC" "C25741"
+		(property "LCSC" "C25765"
 			(at 256.54 205.74 0)
 			(effects
@@
 			)
 		)
-		(property "Value" "39k"
+		(property "Value" "33k"
 			(at 124.46 100.33 0)
 			(effects
@@
 			)
 		)
-		(property "Description" "String R2 (39k + 3.9k)"
+		(property "Description" "String R2 (33k + 10k)"
 			(at 127 99.06 0)
 			(effects
@@
 			)
 		)
-		(property "LCSC" "C25783"
+		(property "LCSC" "C25779"
 			(at 127 99.06 0)
 			(effects
@@
 			)
 		)
-		(property "Footprint" "Resistor_SMD:R_0402_1005Metric"
+		(property "Footprint" "Resistor_SMD:R_0603_1608Metric"
 			(at 127 124.46 0)
 			(effects
@@
 			)
 		)
-		(property "LCSC" "C25755"
+		(property "LCSC" "C22807"
 			(at 127 124.46 0)
 			(effects
@@
 			)
 		)
-		(property "Value" "100k"
+		(property "Value" "20k"
 			(at 45.72 207.01 0)
 			(effects
@@
 			)
 		)
-		(property "LCSC" "C25741"
+		(property "LCSC" "C25765"
 			(at 48.26 205.74 0)
 			(effects
@@
 		(in_bom yes)
 		(on_board yes)
-		(dnp yes)
+		(dnp no)
 		(property "Reference" "R115"
 			(at 147.32 217.17 0)
@@
 			)
 		)
-		(property "Value" "1M"
+		(property "Value" "150k"
 			(at 147.32 219.71 0)
 			(effects
@@
 			)
 		)
-		(property "Description" "Trim, DNP"
+		(property "Description" "FB R2 (R114 33k || 150k)"
 			(at 149.86 218.44 0)
 			(effects
@@
 			)
 		)
-		(property "LCSC" ""
+		(property "LCSC" "C22807"
 			(at 149.86 218.44 0)
 			(effects
@@
 			)
 		)
-		(property "Fit" "DNP"
+		(property "Fit" "JLC"
 			(at 149.86 218.44 0)
 			(effects
@@
 			)
 		)
-		(property "Value" "100k"
+		(property "Value" "51k"
 			(at 238.76 90.17 0)
 			(effects
@@
 			)
 		)
-		(property "LCSC" "C25741"
+		(property "LCSC" "C25794"
 			(at 241.3 88.9 0)
 			(effects
