File: pcb/5-io.kicad_sch (KiCad schematic)
At the start: 0 parts

Commit message: Phase 3: populate io sheet
TCA9555 expander (0x20) with I2C pull-ups and a pin table, five LEDs
(status yellow, activity red, spare red/yellow/green on P05-P07; the
green gets 470R), microSD socket with SDIO pull-ups, and test pads for
the rails, TERMPWR_EN, the expander INT and spare pins P15-P17.

Generator: inline power symbols for dense connectors (the netlist
check caught a rail dogleg shorting SD_CMD and SD_D0).

Co-Authored-By: Claude Opus 5.5 <noreply@anthropic.com>
Parts:
- added C501, C503: 100nF, Capacitor_SMD:C_0402_1005Metric, symbol Device:C
- added C502: 10uF 25V, Capacitor_SMD:C_0805_2012Metric, symbol Device:C
- added D501, D504: KT-0805Y yellow, LED_SMD:LED_0805_2012Metric, symbol Device:LED
- added D502, D503: KT-0603R red, LED_SMD:LED_0603_1608Metric, symbol Device:LED
- added D505: KT-0805G green, LED_SMD:LED_0805_2012Metric, symbol Device:LED
- added J501: TF PUSH, symbol Connector:Micro_SD_Card_Det1
- added R501, R502: 4.7k, Resistor_SMD:R_0402_1005Metric, symbol Device:R
- added R503, R506, R507, R508, R509, R510: 10k, Resistor_SMD:R_0402_1005Metric, symbol Device:R
- added R504, R505, R511, R512: 1k, Resistor_SMD:R_0402_1005Metric, symbol Device:R
- added R513: 470R, Resistor_SMD:R_0402_1005Metric, symbol Device:R
- added TP501: INT, TestPoint:TestPoint_Pad_D1.5mm, symbol Connector:TestPoint
- added TP502: +5V_SYS, TestPoint:TestPoint_Pad_D1.5mm, symbol Connector:TestPoint
- added TP503: +3V3, TestPoint:TestPoint_Pad_D1.5mm, symbol Connector:TestPoint
- added TP504: VTERM, TestPoint:TestPoint_Pad_D1.5mm, symbol Connector:TestPoint
- added TP505: TERMPWR, TestPoint:TestPoint_Pad_D1.5mm, symbol Connector:TestPoint
- added TP506: TP_EN, TestPoint:TestPoint_Pad_D1.5mm, symbol Connector:TestPoint
- added TP507: GND, TestPoint:TestPoint_Pad_D1.5mm, symbol Connector:TestPoint
- added TP508: P15, TestPoint:TestPoint_Pad_D1.5mm, symbol Connector:TestPoint
- added TP509: P16, TestPoint:TestPoint_Pad_D1.5mm, symbol Connector:TestPoint
- added TP510: P17, TestPoint:TestPoint_Pad_D1.5mm, symbol Connector:TestPoint
- added U501: TCA9555PWR, Package_SO:TSSOP-24_4.4x7.8mm_P0.65mm, symbol Interface_Expansion:TCA9555PWR
Connections:
- net BENCH_EFUSE_FAULT_INVERTED: now also U501.7 (P03)
- net FT232H_RESET_INVERTED: now also U501.16 (P13)
- net HUB_RESET_INVERTED: now also U501.17 (P14)
- net I2C_SCL: now also R502.2, U501.22 (SCL)
- net I2C_SDA: now also R501.2, U501.23 (SDA)
- net IS_BENCH_POWERED: now also U501.6 (P02)
- net SD_CLK: now also J501.5 (CLK)
- net SD_CMD: now also J501.3 (CMD), R506.2
- net SD_D0: now also J501.7 (DAT0), R507.2
- net TERMINATOR_EN_INVERTED_FIRMWARE: now also U501.15 (P12)
- net TERMPWR_EFUSE_FAULT_INVERTED: now also U501.8 (P04)
- net TERMPWR_EN_INVERTED: now also TP506.1, U501.5 (P01)
- new net: D505.2 (A), R513.2
- new net: D501.2 (A), R504.2
- new net: D502.2 (A), R505.2
- new net: D503.2 (A), R511.2
- new net: D504.2 (A), R512.2
- new net +3V3: C501.1, C502.1, C503.1, J501.4 (VDD), R501.1, R502.1, R503.1, R504.1, R505.1, R506.1, R507.1, R508.1, R509.1, R510.1, R511.1, R512.1, R513.1, TP503.1, U501.24 (VCC)
- new net +5V_SYS: TP502.1
- new net EXPANDER_INTERRUPT_INVERTED: R503.2, TP501.1, U501.1 (~{INT})
- new net EXPANDER_P15: TP508.1, U501.18 (P15)
- new net EXPANDER_P16: TP509.1, U501.19 (P16)
- new net EXPANDER_P17: TP510.1, U501.20 (P17)
- new net GND: C501.2, C502.2, C503.2, J501.10 (SHIELD), J501.6 (VSS), TP507.1, U501.12 (GND), U501.2 (A1), U501.21 (A0), U501.3 (A2)
- new net LED_ACTIVITY_INVERTED: D502.1 (K), U501.14 (P11)
- new net LED_GREEN_INVERTED: D505.1 (K), U501.11 (P07)
- new net LED_RED_INVERTED: D503.1 (K), U501.9 (P05)
- new net LED_STATUS_INVERTED: D501.1 (K), U501.13 (P10)
- new net LED_YELLOW_INVERTED: D504.1 (K), U501.10 (P06)
- new net SD_CARD_DETECT: J501.9 (DET), U501.4 (P00)
- new net SD_D1: J501.8 (DAT1), R508.2
- new net SD_D2: J501.1 (DAT2), R509.2
- new net SD_D3: J501.2 (DAT3/CD), R510.2
- new net TERMPWR: TP505.1
- new net VTERMINATOR: TP504.1
Other:
- note added: "1k: ~1.3 mA red/yellow. Green (KT-0805G, Vf 2.6-3.1 V at 5 mA) gets 470R: ~2.4 V at low current, so ~1.8 mA typical, >= ~0.7 mA at the top of the Vf spread."
- note added: "Bare pads for probing at bring-up (not on the BOM). P15-P17: spare expander pins; INT: the expander interrupt (firmware polls, so it goes nowhere else)."
- note added: "FT232H_3V3 gets its own pad on the ft232h sheet."
- note added: "I/O expander (TCA9555, I2C0 address 0x20)"
- note added: "LEDs"
- note added: "Lit when the expander drives the pin low. P05-P07: spare, use decided in firmware."
- note added: "Pull-ups 10k (SD spec: 10-100k) on CMD and D0-D3. D3 doubles as card detect in SPI mode; we use the socket's switch instead (DET -> P00). Unverified: DET pin number and switch polarity (LCSC datasheet wasn't downloadable by script). Check before drawing the footprint."
- note added: "Slow signals: status in on port 0, controls out on port 1 (our convention; every pin has its own direction bit). All pins power up as inputs with ~100k pull-ups, so the board is safe with no firmware."
- note added: "Spill-over storage when the host stalls. CLK, CMD, D0 go to the RP2350 (through the rework links); D1-D3 are only pulled up."
- note added: "Test points"
- note added: "microSD (1-bit SDIO on PIO2)"
- note removed: "I/O (blocks/5-rp2350-pinout.md, TCA9555 section) TCA9555 expander (0x20) + 4.7 k I²C pull-ups, INT test point, microSD socket + SDIO pull-ups + 10 µF/100 nF, LED1/LED2, board test points."
