File: pcb/5-io.kicad_sch (KiCad schematic)
At the start: 33 parts, among them J501 TF PUSH, U501 TCA9555PWR

Commit message: all routed
Connections:
- net LED_ACTIVITY_INVERTED: no longer U501.14 (P11)
- net LED_RED_INVERTED: no longer U501.13 (P10)
- net LED_YELLOW_INVERTED: no longer U501.11 (P07)
- net SD_CARD_DETECT: now also U501.13 (P10)
- new net BENCH_EFUSE_FAULT_INVERTED: U501.11 (P07)
- new net IS_BENCH_POWERED: U501.14 (P11)
Other:
- note added: "Lit when the expander drives the pin low. P02-P04: spare, use decided in firmware."
- note added: "Pull-ups 10k (SD spec: 10-100k) on CMD and D0-D3. D3 doubles as card detect in SPI mode; we use the socket's switch instead (DET -> P10). DET = the drawing's 'Cd' pad; it switches against the shell (GND). P10's internal pull-up (TCA9555) is the only pull-up. Polarity (closed with or without a card) isn't on the drawing: check at bring-up."
- note added: "Slow signals: inputs and outputs are mixed across both ports to suit the routing (every pin has its own direction bit; see the table). All pins power up as inputs with ~100k pull-ups, so the board is safe with no firmware."
- note removed: "Lit when the expander drives the pin low. P05-P07: spare, use decided in firmware."
- note removed: "Pull-ups 10k (SD spec: 10-100k) on CMD and D0-D3. D3 doubles as card detect in SPI mode; we use the socket's switch instead (DET -> P00). DET = the drawing's 'Cd' pad; it switches against the shell (GND). P00's internal pull-up (TCA9555) is the only pull-up. Polarity (closed with or without a card) isn't on the drawing: check at bring-up."
- note removed: "Slow signals: status in on port 0, controls out on port 1 (our convention; every pin has its own direction bit). All pins power up as inputs with ~100k pull-ups, so the board is safe with no firmware."
Changed lines of the file:
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@@
 		)
 	)
-	(text "Pull-ups 10k (SD spec: 10-100k) on CMD and D0-D3. D3 doubles as\ncard detect in SPI mode; we use the socket's switch instead (DET -> P00).\nDET = the drawing's 'Cd' pad; it switches against the shell (GND).\nP00's internal pull-up (TCA9555) is the only pull-up. Polarity\n(closed with or without a card) isn't on the drawing: check at bring-up."
+	(text "Pull-ups 10k (SD spec: 10-100k) on CMD and D0-D3. D3 doubles as\ncard detect in SPI mode; we use the socket's switch instead (DET -> P10).\nDET = the drawing's 'Cd' pad; it switches against the shell (GND).\nP10's internal pull-up (TCA9555) is the only pull-up. Polarity\n(closed with or without a card) isn't on the drawing: check at bring-up."
 		(exclude_from_sim no)
 		(at 266.7 160.02 0)
@@
 		)
 	)
-	(text "Slow signals: status in on port 0, controls out on port 1 (our convention; every pin has its own\ndirection bit). All pins power up as inputs with ~100k pull-ups, so the board is safe with no firmware."
+	(text "Slow signals: inputs and outputs are mixed across both ports to suit the routing (every pin has\nits own direction bit; see the table). All pins power up as inputs with ~100k pull-ups, so the board is safe with no firmware."
 		(exclude_from_sim no)
 		(at 20.32 24.82 0)
@@
 		)
 	)
-	(text "Lit when the expander drives the pin low. P05-P07: spare, use decided in firmware."
+	(text "Lit when the expander drives the pin low. P02-P04: spare, use decided in firmware."
 		(exclude_from_sim no)
 		(at 20.32 215.32 0)
@@
 				)
 			)
-			(table_cell "P00 in"
+			(table_cell "P00/P07 in"
 				(exclude_from_sim no)
 				(at 20.32 153.035 0)
@@
 				)
 			)
-			(table_cell "SD_CARD_DETECT"
+			(table_cell "*_EFUSE_FAULT_INVERTED"
 				(exclude_from_sim no)
 				(at 43.18 153.035 0)
@@
 				)
 			)
-			(table_cell "microSD card switch (Cd to shell/GND; polarity: check at bring-up)"
+			(table_cell "low = TERMPWR (P00) / bench (P07) eFuse fault (or reverse block)"
 				(exclude_from_sim no)
 				(at 104.14 153.035 0)
@@
 				)
 			)
-			(table_cell "P02 in"
+			(table_cell "P02-P04 out"
 				(exclude_from_sim no)
 				(at 20.32 161.925 0)
@@
 				)
 			)
-			(table_cell "IS_BENCH_POWERED"
+			(table_cell "LED_GREEN/YELLOW/RED_INVERTED"
 				(exclude_from_sim no)
 				(at 43.18 161.925 0)
@@
 				)
 			)
-			(table_cell "high = running on the bench input (TPS2116 ST)"
+			(table_cell "spare LEDs (green, yellow, red); use to be decided in firmware"
 				(exclude_from_sim no)
 				(at 104.14 161.925 0)
@@
 				)
 			)
-			(table_cell "P03/P04 in"
+			(table_cell "P05/P06 out"
 				(exclude_from_sim no)
 				(at 20.32 166.37 0)
@@
 				)
 			)
-			(table_cell "*_EFUSE_FAULT_INVERTED"
+			(table_cell "LED_ACTIVITY/STATUS_INVERTED"
 				(exclude_from_sim no)
 				(at 43.18 166.37 0)
@@
 				)
 			)
-			(table_cell "low = bench / TERMPWR eFuse fault (or reverse block)"
+			(table_cell "drive low to light the activity (red) / status (yellow) LED"
 				(exclude_from_sim no)
 				(at 104.14 166.37 0)
@@
 				)
 			)
-			(table_cell "P05-P07 out"
+			(table_cell "P10 in"
 				(exclude_from_sim no)
 				(at 20.32 170.815 0)
@@
 				)
 			)
-			(table_cell "LED_RED/YELLOW/GREEN_INVERTED"
+			(table_cell "SD_CARD_DETECT"
 				(exclude_from_sim no)
 				(at 43.18 170.815 0)
@@
 				)
 			)
-			(table_cell "spare LEDs (red, yellow, green); use to be decided in firmware"
+			(table_cell "microSD card switch (Cd to shell/GND; polarity: check at bring-up)"
 				(exclude_from_sim no)
 				(at 104.14 170.815 0)
@@
 				)
 			)
-			(table_cell "P10/P11 out"
+			(table_cell "P11 in"
 				(exclude_from_sim no)
 				(at 20.32 175.26 0)
@@
 				)
 			)
-			(table_cell "LED_STATUS/ACTIVITY_INVERTED"
+			(table_cell "IS_BENCH_POWERED"
 				(exclude_from_sim no)
 				(at 43.18 175.26 0)
@@
 				)
 			)
-			(table_cell "drive low to light the status (yellow) / activity (red) LED"
+			(table_cell "high = running on the bench input (TPS2116 ST)"
 				(exclude_from_sim no)
 				(at 104.14 175.26 0)
@@
 		)
 	)
-	(label "LED_ACTIVITY_INVERTED"
+	(hierarchical_label "IS_BENCH_POWERED"
+		(shape input)
 		(at 160.02 109.22 0)
 		(effects
@@
 				(size 1.27 1.27)
 			)
-			(justify left bottom)
-		)
-	)
-	(label "TERMPWR_EFUSE_FAULT_INVERTED"
+			(justify left)
+		)
+	)
+	(hierarchical_label "TERMPWR_EFUSE_FAULT_INVERTED"
+		(shape input)
 		(at 160.02 83.82 0)
 		(effects
@@
 				(size 1.27 1.27)
 			)
-			(justify left bottom)
+			(justify left)
 		)
 	)
@@
 		)
 	)
-	(label "LED_YELLOW_INVERTED"
+	(hierarchical_label "BENCH_EFUSE_FAULT_INVERTED"
+		(shape input)
 		(at 160.02 101.6 0)
 		(effects
@@
 				(size 1.27 1.27)
 			)
-			(justify left bottom)
+			(justify left)
 		)
 	)
@@
 		)
 	)
-	(label "LED_RED_INVERTED"
+	(label "SD_CARD_DETECT"
 		(at 160.02 106.68 0)
 		(effects
@@
 		)
 	)
-	(hierarchical_label "LED_GREEN_INVERTED"
-		(shape input)
+	(label "LED_GREEN_INVERTED"
 		(at 160.02 88.9 0)
 		(effects
@@
 				(size 1.27 1.27)
 			)
-			(justify left)
+			(justify left bottom)
 		)
 	)
@@
 		)
 	)
-	(hierarchical_label "LED_RED_INVERTED"
-		(shape input)
+	(label "LED_RED_INVERTED"
 		(at 160.02 93.98 0)
 		(effects
@@
 				(size 1.27 1.27)
 			)
-			(justify left)
+			(justify left bottom)
 		)
 	)
@@
 		)
 	)
-	(hierarchical_label "LED_YELLOW_INVERTED"
-		(shape input)
+	(label "LED_YELLOW_INVERTED"
 		(at 160.02 91.44 0)
 		(effects
@@
 				(size 1.27 1.27)
 			)
-			(justify left)
-		)
-	)
+			(justify left bottom)
+		)
+	)
