File: pcb/6-usb-hub.kicad_sch (KiCad schematic)
At the start: 0 parts

Commit message: Phase 3: populate USB-C and hub sheet
USB-C receptacle (both D+/D- pins tied, 5.1k Rd on CC, shell through
0R), ESD on D+/D-, CC and VBUS, and the CH334P hub (new project
symbol from the English datasheet) in external 3.3 V mode: port 1 to
the FT232H, port 2 to the RP2350, reset through a Schottky, crystal
with unfitted load-cap pads, and a "hub active" LED on PGANG.

Net-class patterns simplified to *USB_D+/- and *USB_FT_D+/-:
kicad-cli's netlist only applies patterns to root-level hierarchical
nets, but pcbnew resolves these correctly (checked with its Python API).

Co-Authored-By: Claude Opus 5.5 <noreply@anthropic.com>
Parts:
- added C601: 10uF 25V, Capacitor_SMD:C_0805_2012Metric, symbol Device:C
- added C602, C603: 100nF, Capacitor_SMD:C_0402_1005Metric, symbol Device:C
- added C604, C605: DNP, Capacitor_SMD:C_0402_1005Metric, symbol Device:C
- added D601, D602: H5VUD5BB, Diode_SMD:D_SOD-523, symbol Device:D_TVS
- added D603, D604: H7VL10B, Diode_SMD:D_0402_1005Metric, symbol Device:D_TVS
- added D605: SMF6.0A, Diode_SMD:D_SMF, symbol Device:D_Zener
- added D606: 1N5819WS, Diode_SMD:D_SOD-323, symbol Device:D_Schottky
- added D607: KT-0805G green, LED_SMD:LED_0805_2012Metric, symbol Device:LED
- added J601: USB-C (HRO TYPE-C-31-M-12), Connector_USB:USB_C_Receptacle_HRO_TYPE-C-31-M-12, symbol Connector:USB_C_Receptacle_USB2.0_16P
- added R601, R602: 5.1k, Resistor_SMD:R_0402_1005Metric, symbol Device:R
- added R603: 0R, Resistor_SMD:R_0402_1005Metric, symbol Device:R
- added R604: 470R, Resistor_SMD:R_0402_1005Metric, symbol Device:R
- added U601: CH334P, Package_DFN_QFN:QFN-16-1EP_3x3mm_P0.5mm_EP1.75x1.75mm, symbol scsi-adapter:CH334P
- added Y601: 12MHz ABM8-272-T3, Crystal:Crystal_SMD_3225-4Pin_3.2x2.5mm, symbol Device:Crystal_GND24
Connections:
- net CC1: now also D603.1 (A1), J601.A5 (CC1), R601.1
- net CC2: now also D604.1 (A1), J601.B5 (CC2), R602.1
- net HUB_RESET_INVERTED: now also D606.1 (K)
- net USB_FT_D+: now also U601.10 (DP1)
- net USB_FT_D-: now also U601.9 (DM1)
- net USB_RP_D+: now also U601.8 (DP2)
- net USB_RP_D-: now also U601.7 (DM2)
- net VBUS: now also D605.1 (K), J601.A4 (VBUS), J601.A9 (VBUS), J601.B4 (VBUS), J601.B9 (VBUS)
- new net: D607.2 (A), R604.2
- new net: J601.S1 (SHIELD), R603.1
- new net: D606.2 (A), U601.13 (~{RESET}/CDP)
- new net +3V3: C601.1, C602.1, C603.1, R604.1, U601.15 (V5), U601.16 (VDD33)
- new net GND: C601.2, C602.2, C603.2, C604.2, C605.2, D601.2 (A2), D602.2 (A2), D603.2 (A2), D604.2 (A2), D605.2 (A), J601.A1 (GND), J601.A12 (GND), J601.B1 (GND), J601.B12 (GND), R601.2, R602.2, R603.2, U601.17 (GND), Y601.2 (G), Y601.4 (G)
- new net HUB_ACTIVE_INVERTED: D607.1 (K), U601.14 (PGANG)
- new net HUB_XI: C604.1, U601.2 (XI), Y601.1
- new net HUB_XO: C605.1, U601.1 (XO), Y601.3
- new net USB_D+: D601.1 (A1), J601.A6 (D+), J601.B6 (D+), U601.12 (DPU)
- new net USB_D-: D602.1 (A1), J601.A7 (D-), J601.B7 (D-), U601.11 (DMU)
- no-connect marks 0 -> 6
Other:
- note added: "Both D+ pins and both D- pins are tied, so the plug works either way round. SBU unused. 5.1k Rd on each CC makes us a sink; the CC voltage tells the TERMPWR sheet the port's current."
- note added: "C604/C605 DNP: the CH334 has ~16 pF on each pin (datasheet V2.91 6.1), which suits the ABM8's CL 10 pF. Fit only if the oscillator is off-frequency or slow to start."
- note added: "Clamp static from the cable or a finger to GND before it reaches the hub or the CC comparators. D+/D-: H5VUD5BB, 0.3 pF (fine at 480 Mbit/s). CC: H7VL10B, 7 V working (CC can sit near 5.5 V). VBUS: SMF6.0A, above VBUS's 5.5 V max. Place all five right at the receptacle."
- note added: "D603/D604 are DFN1006 (1.0 x 0.6 mm); the 0402 footprint is a stand-in to check."
- note added: "ESD at the connector"
- note added: "External 3.3 V mode: V5 and VDD33 both on +3V3 (its low-voltage reset can trip as high as 3.2 V, so no internal LDO). Known flaw: no VBUS sense, so on the bench supply with the host off, the 1.5k D+ pull-up back-drives the host. Switch the bench off first."
- note added: "Hub active: lit while the hub isn't suspended."
- note added: "PGANG ('power gang': on bigger CH334 packages it selects ganged port power and overcurrent control; our reading, WCH doesn't spell it out). Its internal pull-up keeps the default mode at reset; afterwards it outputs low while the hub is active, high in suspend. D607 is the 'hub active' LED on it (datasheet 3.3.5, Fig. 3-3-5 left)."
- note added: "Ports 3 and 4 unused (built-in pull-downs; leave open)."
- note added: "RESET#: no external pull-up. The internal ~25k means 'run'; a pin driven high at power-up would enable CDP charging and turn off hub sleep (WCH). The expander (P14) can only pull it low, via D606."
- note added: "Shell: 0R to GND (R603). Swap for 1M || 4.7 nF if EMC testing wants the shield separated from GND."
- note added: "USB 2.0 hub (CH334P)"
- note added: "USB-C receptacle (USB 2.0)"
- note added: "Upstream from the USB-C; port 1 -> FT232H (high speed, the scan data), port 2 -> RP2350 native USB (full speed: updates and console). The hub's transaction translators keep port 1 at full HS bandwidth. USB_D+/- and USB_FT_D+/- are 90R pairs (net class USB_HS); each segment <= ~15 mm."
- note removed: "USB-C and hub (blocks/4-usb.md) USB-C receptacle (HRO TYPE-C-31-M-12), 5.1 k Rd ×2, shell 0 Ω, CC/D±/VBUS ESD, CH334P hub (external 3.3 V) + 12 MHz crystal, 1N5819WS reset diode. USB_D± (connector-hub) and USB_FT_D± are 90 Ω pairs: net class USB_HS, each segment ≤ 15 mm."
