File: pcb/4-rp2350.kicad_sch (KiCad schematic)
At the start: 61 parts, among them J401 TC2030-IDC, SW401 BOOTSEL, SW402 RUN, U401 RP2350B, U402 W25Q128JVSIQ, U403 APS6404L-3SQR-SN, Y401 12MHz ABM8-272-T3

Commit message: basic pcb layout
Parts:
- C402, C403: footprint Capacitor_SMD:C_0402_1005Metric -> scsi-adapter:C_0402_1005Metric_Wide
Changed lines of the file:
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@@
 		(property "Reference" "C402" (at 22.86 87.63 0) (effects (font (size 1.27 1.27)) (justify right)))
 		(property "Value" "4.7uF 10V" (at 22.86 90.17 0) (effects (font (size 1.27 1.27)) (justify right)))
-		(property "Footprint" "Capacitor_SMD:C_0402_1005Metric" (at 25.4 88.9 0) (effects (font (size 1.27 1.27)) (hide yes)))
+		(property "Footprint" "scsi-adapter:C_0402_1005Metric_Wide" (at 25.4 88.9 0) (effects (font (size 1.27 1.27)) (hide yes)))
 		(property "Datasheet" "" (at 25.4 88.9 0) (effects (font (size 1.27 1.27)) (hide yes)))
 		(property "Description" "CIN at VREG_VIN (pin 64)" (at 25.4 88.9 0) (effects (font (size 1.27 1.27)) (hide yes)))
@@
 		(property "Reference" "C403" (at 43.18 87.63 0) (effects (font (size 1.27 1.27)) (justify right)))
 		(property "Value" "4.7uF 10V" (at 43.18 90.17 0) (effects (font (size 1.27 1.27)) (justify right)))
-		(property "Footprint" "Capacitor_SMD:C_0402_1005Metric" (at 45.72 88.9 0) (effects (font (size 1.27 1.27)) (hide yes)))
+		(property "Footprint" "scsi-adapter:C_0402_1005Metric_Wide" (at 45.72 88.9 0) (effects (font (size 1.27 1.27)) (hide yes)))
 		(property "Datasheet" "" (at 45.72 88.9 0) (effects (font (size 1.27 1.27)) (hide yes)))
 		(property "Description" "COUT at VREG_FB/DVDD" (at 45.72 88.9 0) (effects (font (size 1.27 1.27)) (hide yes)))

Commit message: pin reassignments
Connections:
- net FT232H_MIOSIO2: now also R409.1; no longer R409.2
- net FT232H_MIOSIO3: now also R410.1; no longer R410.2
- net FT232H_MISO: now also R413.2; no longer R413.1
- net FT232H_SCLK: now also R411.2; no longer R411.1
- net FT232H_SS_N: now also R412.2; no longer R412.1
- net LOGIC_ANALYZER_MARKER0: now also R414.2; no longer R414.1
- net LOGIC_ANALYZER_MARKER1: now also R415.2; no longer R415.1
- net at U401.40 (GPIO32): now also R415.1; no longer R407.1
- net at U401.42 (GPIO33): now also R414.1; no longer R408.1
- net GPIO34: now reaches U401.43 (GPIO34)
- net GPIO34: now also R426.1, R427.1; no longer R409.1
- net at U401.44 (GPIO35): now also R413.1; no longer R410.1
- net at U401.52 (GPIO41/ADC1): now also R410.2; no longer R411.2
- net GPIO42: now reaches U401.53 (GPIO42/ADC2)
- net GPIO42: now also R418.1, R419.1; no longer R412.2
- net GPIO43: now reaches U401.54 (GPIO43/ADC3)
- net GPIO43: now also R420.1, R421.1; no longer R413.2
- net GPIO44: now reaches U401.55 (GPIO44/ADC4)
- net GPIO44: now also R422.1, R423.1; no longer R414.2
- net GPIO45: now reaches U401.56 (GPIO45/ADC5)
- net GPIO45: now also R424.1, R425.1; no longer R415.2
- removed net GPIO36: R418.1, R419.1, U401.45 (GPIO36)
- removed net GPIO37: R420.1, R421.1, U401.46 (GPIO37)
- removed net GPIO38: R422.1, R423.1, U401.47 (GPIO38)
- removed net GPIO39: R424.1, R425.1, U401.48 (GPIO39)
- removed net GPIO40: R426.1, R427.1, U401.49 (GPIO40/ADC0)
- new net: R412.1, U401.45 (GPIO36)
- new net: R411.1, U401.46 (GPIO37)
- new net: R407.1, U401.47 (GPIO38)
- new net: R408.1, U401.48 (GPIO39)
- new net: R409.2, U401.49 (GPIO40/ADC0)
Other:
- note added: "Fitted 0R: GPIO 42-45 and 34 -> I2C / microSD (normal). Unfitted 0R: the same GPIO -> FT232H pins 17-20, 27. Moving the links trades I2C + microSD for 8-bit FT1248 (42-45) or 245-FIFO mode (42-45 and 34)."
- note added: "I2C1 SCL / rework D5"
- note added: "I2C1 SDA / rework D4"
- note added: "SD CLK / rework D6"
- note added: "SD CMD / rework D7"
- note added: "SD D0 / rework WR#"
- note removed: "Fitted 0R: GPIO 36-40 -> I2C / microSD (normal). Unfitted 0R: the same GPIO -> FT232H pins 17-20, 27. Moving the links trades I2C + microSD for 8-bit FT1248 (36-39) or 245-FIFO mode (36-40)."
- note removed: "I2C0 SCL (rework: FT232H_D5)"
- note removed: "I2C0 SDA (rework: FT232H_D4)"
- note removed: "microSD CLK (rework: FT232H_D6)"
- note removed: "microSD CMD (rework: FT232H_D7)"
- note removed: "microSD D0 (rework: FT232H_WRITE_INVERTED)"

Commit message: start routing ft232h
Parts:
- R419, R421, R423, R425, R427: footprint Resistor_SMD:R_0402_1005Metric -> Resistor_SMD:R_0805_2012Metric; LCSC C17168 -> C17477
Changed lines of the file:
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@@
 		(property "Reference" "R419" (at 44.45 243.84 90) (effects (font (size 1.27 1.27))))
 		(property "Value" "0R" (at 44.45 246.38 90) (effects (font (size 1.27 1.27))))
-		(property "Footprint" "Resistor_SMD:R_0402_1005Metric" (at 44.45 241.3 0) (effects (font (size 1.27 1.27)) (hide yes)))
+		(property "Footprint" "Resistor_SMD:R_0805_2012Metric" (at 44.45 241.3 0) (effects (font (size 1.27 1.27)) (hide yes)))
 		(property "Datasheet" "" (at 44.45 241.3 0) (effects (font (size 1.27 1.27)) (hide yes)))
 		(property "Description" "GPIO42 -> FT232H pin 17 (rework, DNP)" (at 44.45 241.3 0) (effects (font (size 1.27 1.27)) (hide yes)))
-		(property "LCSC" "C17168" (at 44.45 241.3 0) (effects (font (size 1.27 1.27)) (hide yes)))
+		(property "LCSC" "C17477" (at 44.45 241.3 0) (effects (font (size 1.27 1.27)) (hide yes)))
 		(property "Fit" "DNP" (at 44.45 241.3 0) (effects (font (size 1.27 1.27)) (hide yes)))
 		(pin "1")
@@
 		(property "Reference" "R421" (at 102.87 243.84 90) (effects (font (size 1.27 1.27))))
 		(property "Value" "0R" (at 102.87 246.38 90) (effects (font (size 1.27 1.27))))
-		(property "Footprint" "Resistor_SMD:R_0402_1005Metric" (at 102.87 241.3 0) (effects (font (size 1.27 1.27)) (hide yes)))
+		(property "Footprint" "Resistor_SMD:R_0805_2012Metric" (at 102.87 241.3 0) (effects (font (size 1.27 1.27)) (hide yes)))
 		(property "Datasheet" "" (at 102.87 241.3 0) (effects (font (size 1.27 1.27)) (hide yes)))
 		(property "Description" "GPIO43 -> FT232H pin 18 (rework, DNP)" (at 102.87 241.3 0) (effects (font (size 1.27 1.27)) (hide yes)))
-		(property "LCSC" "C17168" (at 102.87 241.3 0) (effects (font (size 1.27 1.27)) (hide yes)))
+		(property "LCSC" "C17477" (at 102.87 241.3 0) (effects (font (size 1.27 1.27)) (hide yes)))
 		(property "Fit" "DNP" (at 102.87 241.3 0) (effects (font (size 1.27 1.27)) (hide yes)))
 		(pin "1")
@@
 		(property "Reference" "R423" (at 44.45 266.7 90) (effects (font (size 1.27 1.27))))
 		(property "Value" "0R" (at 44.45 269.24 90) (effects (font (size 1.27 1.27))))
-		(property "Footprint" "Resistor_SMD:R_0402_1005Metric" (at 44.45 264.16 0) (effects (font (size 1.27 1.27)) (hide yes)))
+		(property "Footprint" "Resistor_SMD:R_0805_2012Metric" (at 44.45 264.16 0) (effects (font (size 1.27 1.27)) (hide yes)))
 		(property "Datasheet" "" (at 44.45 264.16 0) (effects (font (size 1.27 1.27)) (hide yes)))
 		(property "Description" "GPIO44 -> FT232H pin 19 (rework, DNP)" (at 44.45 264.16 0) (effects (font (size 1.27 1.27)) (hide yes)))
-		(property "LCSC" "C17168" (at 44.45 264.16 0) (effects (font (size 1.27 1.27)) (hide yes)))
+		(property "LCSC" "C17477" (at 44.45 264.16 0) (effects (font (size 1.27 1.27)) (hide yes)))
 		(property "Fit" "DNP" (at 44.45 264.16 0) (effects (font (size 1.27 1.27)) (hide yes)))
 		(pin "1")
@@
 		(property "Reference" "R425" (at 102.87 266.7 90) (effects (font (size 1.27 1.27))))
 		(property "Value" "0R" (at 102.87 269.24 90) (effects (font (size 1.27 1.27))))
-		(property "Footprint" "Resistor_SMD:R_0402_1005Metric" (at 102.87 264.16 0) (effects (font (size 1.27 1.27)) (hide yes)))
+		(property "Footprint" "Resistor_SMD:R_0805_2012Metric" (at 102.87 264.16 0) (effects (font (size 1.27 1.27)) (hide yes)))
 		(property "Datasheet" "" (at 102.87 264.16 0) (effects (font (size 1.27 1.27)) (hide yes)))
 		(property "Description" "GPIO45 -> FT232H pin 20 (rework, DNP)" (at 102.87 264.16 0) (effects (font (size 1.27 1.27)) (hide yes)))
-		(property "LCSC" "C17168" (at 102.87 264.16 0) (effects (font (size 1.27 1.27)) (hide yes)))
+		(property "LCSC" "C17477" (at 102.87 264.16 0) (effects (font (size 1.27 1.27)) (hide yes)))
 		(property "Fit" "DNP" (at 102.87 264.16 0) (effects (font (size 1.27 1.27)) (hide yes)))
 		(pin "1")
@@
 		(property "Reference" "R427" (at 44.45 289.56 90) (effects (font (size 1.27 1.27))))
 		(property "Value" "0R" (at 44.45 292.1 90) (effects (font (size 1.27 1.27))))
-		(property "Footprint" "Resistor_SMD:R_0402_1005Metric" (at 44.45 287.02 0) (effects (font (size 1.27 1.27)) (hide yes)))
+		(property "Footprint" "Resistor_SMD:R_0805_2012Metric" (at 44.45 287.02 0) (effects (font (size 1.27 1.27)) (hide yes)))
 		(property "Datasheet" "" (at 44.45 287.02 0) (effects (font (size 1.27 1.27)) (hide yes)))
 		(property "Description" "GPIO34 -> FT232H pin 27 (rework, DNP)" (at 44.45 287.02 0) (effects (font (size 1.27 1.27)) (hide yes)))
-		(property "LCSC" "C17168" (at 44.45 287.02 0) (effects (font (size 1.27 1.27)) (hide yes)))
+		(property "LCSC" "C17477" (at 44.45 287.02 0) (effects (font (size 1.27 1.27)) (hide yes)))
 		(property "Fit" "DNP" (at 44.45 287.02 0) (effects (font (size 1.27 1.27)) (hide yes)))
 		(pin "1")
