File: pcb/3-scsi.kicad_sch (KiCad schematic)
At the start: 75 parts, among them J301 IDC50 box header, J302 HD50 female R/A, J303 2x17 box header, SW301 DIP 2-pos, U301 SN74LVTH245APWR, U302 SN74LVTH245APWR, U303 SN74LVTH245APWR

Commit message: sch update
Parts:
- added C304, C305, C306: 100nF 50V, Capacitor_SMD:C_0402_1005Metric, symbol Device:C
- added C307, C308: 4.7uF 25V, Capacitor_SMD:C_0805_2012Metric, symbol Device:C
Connections:
- net GND: now also C304.2, C305.2, C306.2, C307.2, C308.2
- net TERMPWR: now also C307.1, C308.1
- net VTERMINATOR: now also C304.1, C305.1, C306.1
Other:
- note added: "C307/C308: TERMPWR bulk, one beside each connector's TERMPWR pin (J301.26, J302.38)."
